File: DCDC-40V8A/balance_power.kicad_sch (KiCad schematic)
At the start: 8 parts

Commit message: renumbering
Parts:
- renumbered D9 to D11, D10 to D12, D11 to D13, D12 to D14, D13 to D15, D14 to D16, D15 to D17, D16 to D18
Changed lines of the file:
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@@
 		(dnp no)
 		(fields_autoplaced yes)
-		(property "Reference" "D11"
+		(property "Reference" "D13"
 			(at 82.55 53.3399 90)
 			(show_name no)
@@
 			(project "DCDC-40V8A"
 				(path "/c2f330be-6ca8-4ed0-86db-c2e1bfb68425/c8faf9a2-a06b-4950-bc84-d537bbe92927"
-					(reference "D11")
+					(reference "D13")
 					(unit 1)
 				)
 				(path "/c2f330be-6ca8-4ed0-86db-c2e1bfb68425/fb171ca2-2c26-4c9d-8646-649d698c8bbc"
-					(reference "D19")
+					(reference "D21")
 					(unit 1)
 				)
@@
 		(dnp no)
 		(fields_autoplaced yes)
-		(property "Reference" "D15"
+		(property "Reference" "D17"
 			(at 153.67 53.3399 90)
 			(show_name no)
@@
 			(project "DCDC-40V8A"
 				(path "/c2f330be-6ca8-4ed0-86db-c2e1bfb68425/c8faf9a2-a06b-4950-bc84-d537bbe92927"
-					(reference "D15")
+					(reference "D17")
 					(unit 1)
 				)
 				(path "/c2f330be-6ca8-4ed0-86db-c2e1bfb68425/fb171ca2-2c26-4c9d-8646-649d698c8bbc"
-					(reference "D23")
+					(reference "D25")
 					(unit 1)
 				)
@@
 		(dnp no)
 		(fields_autoplaced yes)
-		(property "Reference" "D16"
+		(property "Reference" "D18"
 			(at 153.67 69.8499 90)
 			(show_name no)
@@
 			(project "DCDC-40V8A"
 				(path "/c2f330be-6ca8-4ed0-86db-c2e1bfb68425/c8faf9a2-a06b-4950-bc84-d537bbe92927"
-					(reference "D16")
+					(reference "D18")
 					(unit 1)
 				)
 				(path "/c2f330be-6ca8-4ed0-86db-c2e1bfb68425/fb171ca2-2c26-4c9d-8646-649d698c8bbc"
-					(reference "D24")
+					(reference "D26")
 					(unit 1)
 				)
@@
 		(dnp no)
 		(fields_autoplaced yes)
-		(property "Reference" "D14"
+		(property "Reference" "D16"
 			(at 135.89 53.3399 90)
 			(show_name no)
@@
 			(project "DCDC-40V8A"
 				(path "/c2f330be-6ca8-4ed0-86db-c2e1bfb68425/c8faf9a2-a06b-4950-bc84-d537bbe92927"
-					(reference "D14")
+					(reference "D16")
 					(unit 1)
 				)
 				(path "/c2f330be-6ca8-4ed0-86db-c2e1bfb68425/fb171ca2-2c26-4c9d-8646-649d698c8bbc"
-					(reference "D22")
+					(reference "D24")
 					(unit 1)
 				)
@@
 		(dnp no)
 		(fields_autoplaced yes)
-		(property "Reference" "D13"
+		(property "Reference" "D15"
 			(at 118.11 53.3399 90)
 			(show_name no)
@@
 			(project "DCDC-40V8A"
 				(path "/c2f330be-6ca8-4ed0-86db-c2e1bfb68425/c8faf9a2-a06b-4950-bc84-d537bbe92927"
-					(reference "D13")
+					(reference "D15")
 					(unit 1)
 				)
 				(path "/c2f330be-6ca8-4ed0-86db-c2e1bfb68425/fb171ca2-2c26-4c9d-8646-649d698c8bbc"
-					(reference "D21")
+					(reference "D23")
 					(unit 1)
 				)
@@
 		(dnp no)
 		(fields_autoplaced yes)
-		(property "Reference" "D12"
+		(property "Reference" "D14"
 			(at 100.33 53.3399 90)
 			(show_name no)
@@
 			(project "DCDC-40V8A"
 				(path "/c2f330be-6ca8-4ed0-86db-c2e1bfb68425/c8faf9a2-a06b-4950-bc84-d537bbe92927"
-					(reference "D12")
+					(reference "D14")
 					(unit 1)
 				)
 				(path "/c2f330be-6ca8-4ed0-86db-c2e1bfb68425/fb171ca2-2c26-4c9d-8646-649d698c8bbc"
-					(reference "D20")
+					(reference "D22")
 					(unit 1)
 				)
@@
 		(dnp no)
 		(fields_autoplaced yes)
-		(property "Reference" "D10"
+		(property "Reference" "D12"
 			(at 64.77 53.3399 90)
 			(show_name no)
@@
 			(project "DCDC-40V8A"
 				(path "/c2f330be-6ca8-4ed0-86db-c2e1bfb68425/c8faf9a2-a06b-4950-bc84-d537bbe92927"
-					(reference "D10")
+					(reference "D12")
 					(unit 1)
 				)
 				(path "/c2f330be-6ca8-4ed0-86db-c2e1bfb68425/fb171ca2-2c26-4c9d-8646-649d698c8bbc"
-					(reference "D18")
+					(reference "D20")
 					(unit 1)
 				)
@@
 		(dnp no)
 		(fields_autoplaced yes)
-		(property "Reference" "D9"
+		(property "Reference" "D11"
 			(at 46.99 53.3399 90)
 			(show_name no)
@@
 			(project "DCDC-40V8A"
 				(path "/c2f330be-6ca8-4ed0-86db-c2e1bfb68425/c8faf9a2-a06b-4950-bc84-d537bbe92927"
-					(reference "D9")
+					(reference "D11")
 					(unit 1)
 				)
 				(path "/c2f330be-6ca8-4ed0-86db-c2e1bfb68425/fb171ca2-2c26-4c9d-8646-649d698c8bbc"
-					(reference "D17")
-					(unit 1)
-				)
+					(reference "D19")
+					(unit 1)
+				)
