File: DCDC-40V8A/diffamps.kicad_sch (KiCad schematic)
At the start: 36 parts, among them U7 TLV9004, U9 TLV9004

Commit message: renumbering
Parts:
- renumbered C41 to C45, C51 to C46, R96 to R105, R98 to R106, R100 to R107, R102 to R108, R104 to R109, R105 to R110, R106 to R111, R107 to R112, R112 to R113, R113 to R114, R114 to R115, R115 to R116, R120 to R117, R121 to R118, R122 to R119, R123 to R120, R128 to R121, R129 to R122, R130 to R123, R131 to R124, R136 to R125, R137 to R126, R138 to R127, R139 to R128, R144 to R129, R145 to R130, R146 to R131, R147 to R132, R152 to R133, R153 to R134, R154 to R135, R155 to R136, U9 to U14, U7 to U14, U7 to U15, U9 to U15
