File: DCDC-40V8A/power_inputs.kicad_sch (KiCad schematic)
At the start: 29 parts, among them Q66 2N7002, Q69 Si7141DP, Q70 Si7141DP, Q71 2N7002, Q72 2N7002, Q73 Si7141DP, Q74 Si7141DP, Q75 2N7002

Commit message: wip before CP deletion
Parts:
- removed Q66, Q71: 2N7002, Package_TO_SOT_SMD:SOT-23, symbol Transistor_FET:2N7002
- removed Q69, Q70: Si7141DP, Package_SO:PowerPAK_SO-8_Single, symbol Transistor_FET:Si7141DP
- removed R164, R201, R202, R204, R205: 220k, Resistor_SMD:R_0402_1005Metric, symbol Device:R
- removed R165: 10k, Resistor_SMD:R_0402_1005Metric, symbol Device:R
- removed R200, R203: 100k, Resistor_SMD:R_0402_1005Metric, symbol Device:R
- removed U14: (no value), Connector_AMASS:AMASS_XT60PW-M_1x02_P7.20mm_Horizontal, symbol DCDC_custom:VDC_XTxx
Connections:
- net VCC: now also D29.2 (A), D30.2 (A)
- net V_LEFT_AUX_OUT: now also D30.1 (K); no longer D29.1 (K)
- net V_RIGHT_AUX_OUT: now also D29.1 (K); no longer D30.1 (K)
- net RAIL_ADC renamed V_EXT_ADC
- net RAIL_EN renamed PWR_EXT_EN
- net V_RAIL renamed V_EXT
- net V_EXT: no longer D29.2 (A), D30.2 (A)
Other:
- moved on the sheet: Q72, Q73, Q74, Q75, R206, R207, R208, R209, R210, R211, R212, R213

Commit message: renumbering
Parts:
- renumbered D29 to D27, D30 to D28, Q73 to Q46, Q74 to Q47, Q72 to Q48, Q75 to Q49, R207 to R169, R210 to R170, R212 to R171, R208 to R172, R211 to R173, R213 to R174, R206 to R175, R209 to R176, U22 to U18, U21 to U19
Changed lines of the file:
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@@
 		(dnp no)
 		(fields_autoplaced yes)
-		(property "Reference" "#PWR090"
+		(property "Reference" "#PWR0146"
 			(at 162.56 46.99 0)
 			(hide yes)
@@
 			(project "DCDC-40V8A"
 				(path "/c2f330be-6ca8-4ed0-86db-c2e1bfb68425/82e88553-6a2b-4207-ade0-f53f84fac1b6"
-					(reference "#PWR090")
+					(reference "#PWR0146")
 					(unit 1)
 				)
@@
 		(dnp no)
 		(fields_autoplaced yes)
-		(property "Reference" "U21"
+		(property "Reference" "U19"
 			(at 151.13 64.77 0)
 			(hide yes)
@@
 			(project "DCDC-40V8A"
 				(path "/c2f330be-6ca8-4ed0-86db-c2e1bfb68425/82e88553-6a2b-4207-ade0-f53f84fac1b6"
-					(reference "U21")
+					(reference "U19")
 					(unit 1)
 				)
@@
 		(dnp no)
 		(fields_autoplaced yes)
-		(property "Reference" "#PWR089"
+		(property "Reference" "#PWR0145"
 			(at 40.64 46.99 0)
 			(hide yes)
@@
 			(project "DCDC-40V8A"
 				(path "/c2f330be-6ca8-4ed0-86db-c2e1bfb68425/82e88553-6a2b-4207-ade0-f53f84fac1b6"
-					(reference "#PWR089")
+					(reference "#PWR0145")
 					(unit 1)
 				)
@@
 		(dnp no)
 		(fields_autoplaced yes)
-		(property "Reference" "Q75"
+		(property "Reference" "Q49"
 			(at 129.54 77.4699 0)
 			(show_name no)
@@
 			(project "DCDC-40V8A"
 				(path "/c2f330be-6ca8-4ed0-86db-c2e1bfb68425/82e88553-6a2b-4207-ade0-f53f84fac1b6"
-					(reference "Q75")
+					(reference "Q49")
 					(unit 1)
 				)
@@
 		(dnp no)
 		(fields_autoplaced yes)
-		(property "Reference" "R212"
+		(property "Reference" "R171"
 			(at 165.1 52.0699 0)
 			(show_name no)
@@
 			(project "DCDC-40V8A"
 				(path "/c2f330be-6ca8-4ed0-86db-c2e1bfb68425/82e88553-6a2b-4207-ade0-f53f84fac1b6"
-					(reference "R212")
+					(reference "R171")
 					(unit 1)
 				)
@@
 		(in_pos_files yes)
 		(dnp no)
-		(property "Reference" "Q74"
+		(property "Reference" "Q47"
 			(at 118.11 36.83 90)
 			(show_name no)
@@
 			(project "DCDC-40V8A"
 				(path "/c2f330be-6ca8-4ed0-86db-c2e1bfb68425/82e88553-6a2b-4207-ade0-f53f84fac1b6"
-					(reference "Q74")
+					(reference "Q47")
 					(unit 1)
 				)
@@
 		(dnp no)
 		(fields_autoplaced yes)
-		(property "Reference" "#PWR0169"
+		(property "Reference" "#PWR0149"
 			(at 109.22 92.71 0)
 			(hide yes)
@@
 			(project "DCDC-40V8A"
 				(path "/c2f330be-6ca8-4ed0-86db-c2e1bfb68425/82e88553-6a2b-4207-ade0-f53f84fac1b6"
-					(reference "#PWR0169")
+					(reference "#PWR0149")
 					(unit 1)
 				)
@@
 		(in_pos_files yes)
 		(dnp no)
-		(property "Reference" "Q73"
+		(property "Reference" "Q46"
 			(at 85.09 36.83 90)
 			(show_name no)
@@
 			(project "DCDC-40V8A"
 				(path "/c2f330be-6ca8-4ed0-86db-c2e1bfb68425/82e88553-6a2b-4207-ade0-f53f84fac1b6"
-					(reference "Q73")
+					(reference "Q46")
 					(unit 1)
 				)
@@
 		(dnp no)
 		(fields_autoplaced yes)
-		(property "Reference" "D29"
+		(property "Reference" "D27"
 			(at 43.18 46.0374 90)
 			(show_name no)
@@
 			(project "DCDC-40V8A"
 				(path "/c2f330be-6ca8-4ed0-86db-c2e1bfb68425/82e88553-6a2b-4207-ade0-f53f84fac1b6"
-					(reference "D29")
+					(reference "D27")
 					(unit 1)
 				)
@@
 		(in_pos_files yes)
 		(dnp no)
-		(property "Reference" "R211"
+		(property "Reference" "R173"
 			(at 128.27 63.4999 0)
 			(show_name no)
@@
 			(project "DCDC-40V8A"
 				(path "/c2f330be-6ca8-4ed0-86db-c2e1bfb68425/82e88553-6a2b-4207-ade0-f53f84fac1b6"
-					(reference "R211")
+					(reference "R173")
 					(unit 1)
 				)
@@
 		(in_pos_files yes)
 		(dnp no)
-		(property "Reference" "R207"
+		(property "Reference" "R169"
 			(at 74.93 48.2601 0)
 			(show_name no)
@@
 			(project "DCDC-40V8A"
 				(path "/c2f330be-6ca8-4ed0-86db-c2e1bfb68425/82e88553-6a2b-4207-ade0-f53f84fac1b6"
-					(reference "R207")
+					(reference "R169")
 					(unit 1)
 				)
@@
 		(dnp no)
 		(fields_autoplaced yes)
-		(property "Reference" "R210"
+		(property "Reference" "R170"
 			(at 128.27 48.2601 0)
 			(show_name no)
@@
 			(project "DCDC-40V8A"
 				(path "/c2f330be-6ca8-4ed0-86db-c2e1bfb68425/82e88553-6a2b-4207-ade0-f53f84fac1b6"
-					(reference "R210")
+					(reference "R170")
 					(unit 1)
 				)
@@
 		(dnp no)
 		(fields_autoplaced yes)
-		(property "Reference" "D30"
+		(property "Reference" "D28"
 			(at 63.5 46.0374 90)
 			(show_name no)
@@
 			(project "DCDC-40V8A"
 				(path "/c2f330be-6ca8-4ed0-86db-c2e1bfb68425/82e88553-6a2b-4207-ade0-f53f84fac1b6"
-					(reference "D30")
+					(reference "D28")
 					(unit 1)
 				)
@@
 		(dnp no)
 		(fields_autoplaced yes)
-		(property "Reference" "#PWR094"
+		(property "Reference" "#PWR0147"
 			(at 40.64 46.99 0)
 			(hide yes)
@@
 			(project "DCDC-40V8A"
 				(path "/c2f330be-6ca8-4ed0-86db-c2e1bfb68425/82e88553-6a2b-4207-ade0-f53f84fac1b6"
-					(reference "#PWR094")
+					(reference "#PWR0147")
 					(unit 1)
 				)
@@
 		(dnp no)
 		(fields_autoplaced yes)
-		(property "Reference" "R213"
+		(property "Reference" "R174"
 			(at 165.1 74.9299 0)
 			(show_name no)
@@
 			(project "DCDC-40V8A"
 				(path "/c2f330be-6ca8-4ed0-86db-c2e1bfb68425/82e88553-6a2b-4207-ade0-f53f84fac1b6"
-					(reference "R213")
+					(reference "R174")
 					(unit 1)
 				)
@@
 		(dnp no)
 		(fields_autoplaced yes)
-		(property "Reference" "U22"
+		(property "Reference" "U18"
 			(at 140.97 64.77 0)
 			(hide yes)
@@
 			(project "DCDC-40V8A"
 				(path "/c2f330be-6ca8-4ed0-86db-c2e1bfb68425/82e88553-6a2b-4207-ade0-f53f84fac1b6"
-					(reference "U22")
+					(reference "U18")
 					(unit 1)
 				)
@@
 		(dnp no)
 		(fields_autoplaced yes)
-		(property "Reference" "Q72"
+		(property "Reference" "Q48"
 			(at 81.28 77.4699 0)
 			(show_name no)
@@
 			(project "DCDC-40V8A"
 				(path "/c2f330be-6ca8-4ed0-86db-c2e1bfb68425/82e88553-6a2b-4207-ade0-f53f84fac1b6"
-					(reference "Q72")
+					(reference "Q48")
 					(unit 1)
 				)
@@
 		(dnp no)
 		(fields_autoplaced yes)
-		(property "Reference" "R206"
+		(property "Reference" "R175"
 			(at 63.5 81.2799 0)
 			(show_name no)
@@
 			(project "DCDC-40V8A"
 				(path "/c2f330be-6ca8-4ed0-86db-c2e1bfb68425/82e88553-6a2b-4207-ade0-f53f84fac1b6"
-					(reference "R206")
+					(reference "R175")
 					(unit 1)
 				)
@@
 		(dnp no)
 		(fields_autoplaced yes)
-		(property "Reference" "#PWR092"
+		(property "Reference" "#PWR0148"
 			(at 60.96 46.99 0)
 			(hide yes)
@@
 			(project "DCDC-40V8A"
 				(path "/c2f330be-6ca8-4ed0-86db-c2e1bfb68425/82e88553-6a2b-4207-ade0-f53f84fac1b6"
-					(reference "#PWR092")
+					(reference "#PWR0148")
 					(unit 1)
 				)
@@
 		(dnp no)
 		(fields_autoplaced yes)
-		(property "Reference" "R209"
+		(property "Reference" "R176"
 			(at 111.76 81.2799 0)
 			(show_name no)
@@
 			(project "DCDC-40V8A"
 				(path "/c2f330be-6ca8-4ed0-86db-c2e1bfb68425/82e88553-6a2b-4207-ade0-f53f84fac1b6"
-					(reference "R209")
+					(reference "R176")
 					(unit 1)
 				)
@@
 		(in_pos_files yes)
 		(dnp no)
-		(property "Reference" "R208"
+		(property "Reference" "R172"
 			(at 80.01 63.4999 0)
 			(show_name no)
@@
 			(project "DCDC-40V8A"
 				(path "/c2f330be-6ca8-4ed0-86db-c2e1bfb68425/82e88553-6a2b-4207-ade0-f53f84fac1b6"
-					(reference "R208")
-					(unit 1)
-				)
+					(reference "R172")
+					(unit 1)
+				)
