File: DCDC-40V8A/DCDC-40V8A.kicad_sch (KiCad schematic)
At the start: 0 parts

Commit message: wip
Parts:
- added J3, J4: Conn_01x09, Connector_PinHeader_2.54mm:PinHeader_1x09_P2.54mm_Horizontal, symbol Connector_Generic:Conn_01x09
Connections:
- net ADC MUX and Discharge A/BAT_0: now also J3.9 (Pin_9)
- net ADC MUX and Discharge A/BAT_1: now also J3.8 (Pin_8)
- net ADC MUX and Discharge A/BAT_2: now also J3.7 (Pin_7)
- net ADC MUX and Discharge A/BAT_3: now also J3.6 (Pin_6)
- net ADC MUX and Discharge A/BAT_4: now also J3.5 (Pin_5)
- net ADC MUX and Discharge A/BAT_5: now also J3.4 (Pin_4)
- net ADC MUX and Discharge A/BAT_6: now also J3.3 (Pin_3)
- net ADC MUX and Discharge A/BAT_7: now also J3.2 (Pin_2)
- net ADC MUX and Discharge A/BAT_8: now also J3.1 (Pin_1)
- net ADC MUX and Discharge B/BAT_0: now also J4.9 (Pin_9)
- net ADC MUX and Discharge B/BAT_1: now also J4.8 (Pin_8)
- net ADC MUX and Discharge B/BAT_2: now also J4.7 (Pin_7)
- net ADC MUX and Discharge B/BAT_3: now also J4.6 (Pin_6)
- net ADC MUX and Discharge B/BAT_4: now also J4.5 (Pin_5)
- net ADC MUX and Discharge B/BAT_5: now also J4.4 (Pin_4)
- net ADC MUX and Discharge B/BAT_6: now also J4.3 (Pin_3)
- net ADC MUX and Discharge B/BAT_7: now also J4.2 (Pin_2)
- net ADC MUX and Discharge B/BAT_8: now also J4.1 (Pin_1)
Other:
- added sheet Balance Power A (balance_power.kicad_sch)
- added sheet Balance Power B (balance_power.kicad_sch)
- added sheet Cell_V_DiffAmps A (diffamps.kicad_sch)
- added sheet Cell_V_DiffAmps B (diffamps.kicad_sch)
- added sheet Power Inputs (power_inputs.kicad_sch)
- added sheet Power Outputs (power_outputs.kicad_sch)
- added sheet Temp Sensors (temp_sensors.kicad_sch)
- sheet ADC MUX and Discharge A ports: added ADC_OUT_L, MEAS_L[1..8]; removed ADC_OUT, MEAS_ADC[1..8]
- sheet ADC MUX and Discharge B ports: added ADC_OUT_L, MEAS_L[1..8]; removed ADC_OUT, MEAS_ADC[1..8]
- sheet ADC-Coprocessor ports: added 5V_DCDC_DIS, BAT_DCDC_DIS, CP_PWM, PWR_RAIL_EN, PWR_XT60IN_EN, VBAT_A_ADC, VBAT_B_ADC, V_RAIL_ADC, V_XT60IN_ADC; removed BAT_5V_DIS, MAIN_5V_DIS, PWR_LEFT_EN, PWR_RIGHT_EN, VBAT_ADC, VCC_ADC
- sheet Power ports: added 5V_DCDC_DIS, BAL_PWR, BAT_DCDC_DIS, CP_PWM, PWR_5V_EN; removed BAT_5V_DIS, MAIN_5V_DIS

Commit message: wip before CP deletion
Other:
- sheet ADC-Coprocessor ports: added PWR_EXT_EN, V_EXT_ADC; removed PWR_RAIL_EN, PWR_XT60IN_EN, V_RAIL_ADC, V_XT60IN_ADC
- sheet Power Inputs ports: added PWR_EXT_EN, V_EXT_ADC; removed RAIL_ADC, RAIL_EN, XT60IN_ADC, XT60IN_EN
Changed lines of the file:
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@@
 	(wire
 		(pts
-			(xy 86.36 124.46) (xy 105.41 124.46)
+			(xy 86.36 128.27) (xy 105.41 128.27)
 		)
 		(stroke
@@
 	(wire
 		(pts
-			(xy 86.36 127) (xy 105.41 127)
-		)
-		(stroke
-			(width 0)
-			(type default)
-		)
-	)
-	(wire
-		(pts
 			(xy 309.88 110.49) (xy 309.88 171.45)
 		)
@@
 	(wire
 		(pts
-			(xy 86.36 129.54) (xy 105.41 129.54)
-		)
-		(stroke
-			(width 0)
-			(type default)
-		)
-	)
-	(wire
-		(pts
 			(xy 154.94 222.25) (xy 154.94 233.68)
 		)
@@
 	(wire
 		(pts
-			(xy 86.36 121.92) (xy 105.41 121.92)
+			(xy 86.36 125.73) (xy 105.41 125.73)
 		)
 		(stroke
@@
 			)
 		)
-		(pin "PWR_RAIL_EN" output
-			(at 105.41 124.46 180)
-			(effects
-				(font
-					(size 1.27 1.27)
-				)
-				(justify left)
-			)
-		)
-		(pin "PWR_XT60IN_EN" output
-			(at 105.41 127 180)
-			(effects
-				(font
-					(size 1.27 1.27)
-				)
-				(justify left)
-			)
-		)
-		(pin "V_RAIL_ADC" input
-			(at 105.41 121.92 180)
-			(effects
-				(font
-					(size 1.27 1.27)
-				)
-				(justify left)
-			)
-		)
-		(pin "V_XT60IN_ADC" input
-			(at 105.41 129.54 180)
+		(pin "PWR_EXT_EN" output
+			(at 105.41 125.73 180)
+			(effects
+				(font
+					(size 1.27 1.27)
+				)
+				(justify left)
+			)
+		)
+		(pin "V_EXT_ADC" input
+			(at 105.41 128.27 180)
 			(effects
 				(font
@@
 	)
 	(sheet
-		(at 33.02 78.74)
-		(size 53.34 64.77)
+		(at 33.02 116.84)
+		(size 53.34 19.05)
 		(exclude_from_sim no)
 		(in_bom yes)
@@
 		)
 		(property "Sheetname" "Power Inputs"
-			(at 33.02 78.0284 0)
+			(at 33.02 116.1284 0)
 			(show_name no)
 			(do_not_autoplace no)
@@
 		)
 		(property "Sheetfile" "power_inputs.kicad_sch"
-			(at 33.02 144.0946 0)
+			(at 33.02 136.4746 0)
 			(show_name no)
 			(do_not_autoplace no)
@@
 			)
 		)
-		(pin "RAIL_ADC" output
-			(at 86.36 121.92 0)
-			(effects
-				(font
-					(size 1.27 1.27)
-				)
-				(justify right)
-			)
-		)
-		(pin "RAIL_EN" input
-			(at 86.36 124.46 0)
-			(effects
-				(font
-					(size 1.27 1.27)
-				)
-				(justify right)
-			)
-		)
-		(pin "XT60IN_ADC" output
-			(at 86.36 129.54 0)
-			(effects
-				(font
-					(size 1.27 1.27)
-				)
-				(justify right)
-			)
-		)
-		(pin "XT60IN_EN" input
-			(at 86.36 127 0)
-			(effects
-				(font
+		(pin "V_EXT_ADC" output
+			(at 86.36 128.27 0)
+			(effects
+				(font
+					(size 1.27 1.27)
+				)
+				(justify right)
+			)
+		)
+		(pin "PWR_EXT_EN" input
+			(at 86.36 125.73 0)
+			(effects
+				(font

Commit message: renumbering
Parts:
- renumbered J3 to J1, J4 to J2
Changed lines of the file:
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@@
 		(dnp no)
 		(fields_autoplaced yes)
-		(property "Reference" "#PWR087"
+		(property "Reference" "#PWR01"
 			(at 312.42 246.38 0)
 			(hide yes)
@@
 			(project "DCDC-40V8A"
 				(path "/c2f330be-6ca8-4ed0-86db-c2e1bfb68425"
-					(reference "#PWR087")
+					(reference "#PWR01")
 					(unit 1)
 				)
@@
 		(dnp no)
 		(fields_autoplaced yes)
-		(property "Reference" "J4"
+		(property "Reference" "J2"
 			(at 393.7 215.8999 0)
 			(show_name no)
@@
 			(project "DCDC-40V8A"
 				(path "/c2f330be-6ca8-4ed0-86db-c2e1bfb68425"
-					(reference "J4")
+					(reference "J2")
 					(unit 1)
 				)
@@
 		(dnp no)
 		(fields_autoplaced yes)
-		(property "Reference" "J3"
+		(property "Reference" "J1"
 			(at 393.7 149.8599 0)
 			(show_name no)
@@
 			(project "DCDC-40V8A"
 				(path "/c2f330be-6ca8-4ed0-86db-c2e1bfb68425"
-					(reference "J3")
+					(reference "J1")
 					(unit 1)
 				)
@@
 			(project "DCDC-40V8A"
 				(path "/c2f330be-6ca8-4ed0-86db-c2e1bfb68425"
-					(page "21")
-				)
-			)
+					(page "5")
+				)
+			)

Commit message: schematics done?
Other:
- added sheet Small External Connectors (conn.kicad_sch)
- sheet ADC-Coprocessor ports: added 12V_EN; removed none
Changed lines of the file:
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@@
 	(wire
 		(pts
-			(xy 86.36 170.18) (xy 105.41 170.18)
+			(xy 86.36 170.18) (xy 104.14 170.18)
 		)
 		(stroke
@@
 	(wire
 		(pts
-			(xy 86.36 128.27) (xy 105.41 128.27)
+			(xy 86.36 128.27) (xy 104.14 128.27)
 		)
 		(stroke
@@
 	(wire
 		(pts
-			(xy 86.36 177.8) (xy 105.41 177.8)
+			(xy 86.36 177.8) (xy 104.14 177.8)
 		)
 		(stroke
@@
 	(wire
 		(pts
-			(xy 86.36 175.26) (xy 105.41 175.26)
+			(xy 86.36 175.26) (xy 104.14 175.26)
 		)
 		(stroke
@@
 	(wire
 		(pts
-			(xy 86.36 172.72) (xy 105.41 172.72)
+			(xy 86.36 172.72) (xy 104.14 172.72)
 		)
 		(stroke
@@
 	(wire
 		(pts
-			(xy 86.36 125.73) (xy 105.41 125.73)
+			(xy 86.36 125.73) (xy 104.14 125.73)
 		)
 		(stroke
@@
 	)
 	(sheet
+		(at 175.26 82.55)
+		(size 48.26 16.51)
+		(exclude_from_sim no)
+		(in_bom yes)
+		(on_board yes)
+		(dnp no)
+		(fields_autoplaced yes)
+		(stroke
+			(width 0.1524)
+			(type solid)
+		)
+		(fill
+			(color 0 0 0 0)
+		)
+		(property "Sheetname" "Small External Connectors"
+			(at 175.26 81.8384 0)
+			(show_name no)
+			(do_not_autoplace no)
+			(effects
+				(font
+					(size 1.27 1.27)
+				)
+				(justify left bottom)
+			)
+		)
+		(property "Sheetfile" "conn.kicad_sch"
+			(at 175.26 99.6446 0)
+			(show_name no)
+			(do_not_autoplace no)
+			(effects
+				(font
+					(size 1.27 1.27)
+				)
+				(justify left top)
+			)
+		)
+		(instances
+			(project "DCDC-40V8A"
+				(path "/c2f330be-6ca8-4ed0-86db-c2e1bfb68425"
+					(page "21")
+				)
+			)
+		)
+	)
+	(sheet
 		(at 123.19 233.68)
 		(size 76.2 22.86)
@@
 	)
 	(sheet
-		(at 105.41 119.38)
-		(size 109.22 102.87)
+		(at 104.14 119.38)
+		(size 110.49 102.87)
 		(exclude_from_sim no)
 		(in_bom yes)
@@
 		)
 		(property "Sheetname" "ADC-Coprocessor"
-			(at 105.41 118.6684 0)
+			(at 104.14 118.6684 0)
 			(show_name no)
 			(do_not_autoplace no)
@@
 		)
 		(property "Sheetfile" "adc_coprocessor.kicad_sch"
-			(at 105.41 222.8346 0)
+			(at 104.14 222.8346 0)
 			(show_name no)
 			(do_not_autoplace no)
@@
 		)
 		(pin "CHAN_A_EN" output
-			(at 105.41 172.72 180)
+			(at 104.14 172.72 180)
 			(effects
 				(font
@@
 		)
 		(pin "CHAN_B_EN" output
-			(at 105.41 175.26 180)
+			(at 104.14 175.26 180)
 			(effects
 				(font
@@
 		)
 		(pin "FAN_EN" output
-			(at 105.41 208.28 180)
+			(at 104.14 208.28 180)
 			(effects
 				(font
@@
 		)
 		(pin "VBAT_A_ADC" input
-			(at 105.41 170.18 180)
+			(at 104.14 170.18 180)
 			(effects
 				(font
@@
 		)
 		(pin "VBAT_B_ADC" input
-			(at 105.41 177.8 180)
+			(at 104.14 177.8 180)
 			(effects
 				(font
@@
 		)
 		(pin "PWR_EXT_EN" output
-			(at 105.41 125.73 180)
+			(at 104.14 125.73 180)
 			(effects
 				(font
@@
 		)
 		(pin "V_EXT_ADC" input
-			(at 105.41 128.27 180)
-			(effects
-				(font
-					(size 1.27 1.27)
-				)
-				(justify left)
+			(at 104.14 128.27 180)
+			(effects
+				(font
+					(size 1.27 1.27)
+				)
+				(justify left)
+			)
+		)
+		(pin "12V_EN" output
+			(at 127 119.38 90)
+			(effects
+				(font
+					(size 1.27 1.27)
+				)
+				(justify right)
 			)
 		)
@@
 	(sheet
 		(at 175.26 24.13)
-		(size 48.26 69.85)
+		(size 48.26 48.26)
 		(exclude_from_sim no)
 		(in_bom yes)
@@
 		)
 		(property "Sheetfile" "control_connector.kicad_sch"
-			(at 175.26 94.5646 0)
+			(at 175.26 72.9746 0)
 			(show_name no)
 			(do_not_autoplace no)
@@
 		)
 		(pin "Left_RX" input
-			(at 175.26 85.09 180)
+			(at 175.26 66.04 180)
 			(effects
 				(font
@@
 		)
 		(pin "Left_TX" output
-			(at 175.26 87.63 180)
+			(at 175.26 68.58 180)
 			(effects
 				(font
@@
 		)
 		(pin "Right_RX" input
-			(at 223.52 85.09 0)
+			(at 223.52 66.04 0)
 			(effects
 				(font
@@
 		)
 		(pin "Right_TX" output
-			(at 223.52 87.63 0)
+			(at 223.52 68.58 0)
 			(effects
 				(font
@@
 	)
 	(sheet
-		(at 106.68 35.56)
-		(size 39.37 57.15)
+		(at 104.14 35.56)
+		(size 41.91 57.15)
 		(exclude_from_sim no)
 		(in_bom yes)
@@
 		)
 		(property "Sheetname" "Power"
-			(at 106.68 34.8484 0)
+			(at 104.14 34.8484 0)
 			(show_name no)
 			(do_not_autoplace no)
@@
 		)
 		(property "Sheetfile" "power.kicad_sch"
-			(at 106.68 93.2946 0)
-			(show_name no)
-			(do_not_autoplace no)
+			(at 104.14 93.2946 0)
+			(show_name no)
+			(do_not_autoplace no)
