File: DCDC-40V8A/power.kicad_sch (KiCad schematic)
At the start: 88 parts, among them Q1 BSS83P, Q10 BSS83P, Q11 2N7002, Q12 2N7002, Q2 2N7002, Q3 2N7002, Q4 2N7002, Q5 CSD18533Q5A, Q6 CSD18533Q5A, Q7 CSD18533Q5A, Q8 CSD18533Q5A, Q9 BSS83P, U1 LGS5145EP, U2 MT3608, U3 GS2019-33TR5

Commit message: schematics done?
Parts:
- added C49: 100u, symbol Device:C_Polarized
- added R193: 100k, Resistor_SMD:R_0603_1608Metric, symbol Device:R
- added R194, R195, R196: 10k, Resistor_SMD:R_0402_1005Metric, symbol Device:R
Connections:
- net +5V: now also Q10.2 (S), C49.1, R195.1; no longer Q10.3 (D), U2.4 (EN)
- net GND: now also C49.2, R193.2
- net VCC: now also Q9.2 (S), R194.1; no longer Q9.3 (D)
- net at Q11.3 (D): now also R196.2; no longer Q9.1 (G)
- net at Q10.1 (G), Q12.3 (D): now also R195.2
- new net: Q9.1 (G), R194.2, R196.1
- new net: Q10.3 (D), Q9.3 (D)
- new net 12V_EN: R193.1, U2.4 (EN)
Other:
- note added: "V_AUX/VCC/V_EXT/VBAT/V_BAL -> 5V Buck (1A)"
- note removed: "V_AUX/VCC/VBAT/V_BAL -> 5V Buck (1A)"
- moved on the sheet: Q10, Q11, Q12, Q9, R27
